File: pcb/esp32_baseboard/esp32_baseboard.kicad_sch (KiCad schematic)
At the start: 23 parts, among them J1 Screw_12V_IN, J10 LIM_MIN_NC, J11 LIM_MAX_NC, J12 LIM_MIN_NC, J13 LIM_MAX_NC, J14 BUP_30S, J17 TFT_TOUCH, J2 NEMA17_OUT, J4 OPTO_FIELD_IN, J5 GA12_N20, J6 GA12_N20, J7 GA12_N20, J8 LIM_MIN_NC, J9 LIM_MAX_NC, U1 ESP32_S3_DevKitC_1, U2 MP1584_5V3A, U3 TMC2209_StepStick, U4 PC817_4CH, U5 DRV8871_Module, U6 DRV8871_Module, U7 DRV8871_Module, U9 PC817_4CH

Commit message: sửa lỗi ngắn mạch trên board
Parts:
- removed J17: TFT_TOUCH, ESP32_Carrier:PinHeader_1x11_TFT, symbol ESP32_Carrier:Conn_1x11_TFT
- added J17: TFT_TOUCH, ESP32_Carrier:PinHeader_1x10_TFT, symbol ESP32_Carrier:Conn_1x10_TFT
- added J18: EC11_ENC, ESP32_Carrier:PinHeader_1x04_ENC, symbol ESP32_Carrier:Conn_1x04_ENC
Connections:
- net +12V: now also J18.1 (GND), J18.2 (3V3)
- net OPTO_OUT6: now also U1.29 (IO41), J18.4 (ENC_B)
- net OPTO_OUT8: no longer names the net of U9.12 (OUT4)
- net OPTO_OUT8: no longer U1.15 (IO9)
- new net: J18.3 (ENC_A), U1.15 (IO9)
Other:
- note added: "J18 ENC: wall-mount EC11 cable → GND/3V3/A/B; CLK=IO9 DT=IO41; no SW"
- note added: "TOP: J2 NEMA17 / J17 TFT / J18 ENC / J15 buzzer / J16 MOSFET"
- note removed: "TOP: J2 NEMA17 phases / J17 TFT / J15 buzzer / J16 MOSFET"
Changed lines of the file:
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@@
 		(effects (font (size 1.27 1.27)) (justify left))
 	)
-	(text "TOP: J2 NEMA17 phases / J17 TFT / J15 buzzer / J16 MOSFET"
+	(text "TOP: J2 NEMA17 / J17 TFT / J18 ENC / J15 buzzer / J16 MOSFET"
 		(at 20.32 120.65 0)
 		(effects (font (size 1.27 1.27)) (justify left))
@@
 		(pin "2")
 		(instances
-			(project "esp32_baseboard" (path "/fea81b1a-a77c-4c77-bfcb-f010ab6c4763" (reference "J1") (unit 1)))
+			(project "esp32_baseboard" (path "/b769966a-c1a5-4e09-8b47-a27c2881840e" (reference "J1") (unit 1)))
 		)
 	)
@@
 		(pin "4")
 		(instances
-			(project "esp32_baseboard" (path "/fea81b1a-a77c-4c77-bfcb-f010ab6c4763" (reference "U2") (unit 1)))
+			(project "esp32_baseboard" (path "/b769966a-c1a5-4e09-8b47-a27c2881840e" (reference "U2") (unit 1)))
 		)
 	)
@@
 		(pin "30")
 		(instances
-			(project "esp32_baseboard" (path "/fea81b1a-a77c-4c77-bfcb-f010ab6c4763" (reference "U1") (unit 1)))
+			(project "esp32_baseboard" (path "/b769966a-c1a5-4e09-8b47-a27c2881840e" (reference "U1") (unit 1)))
 		)
 	)
@@
 		(pin "16")
 		(instances
-			(project "esp32_baseboard" (path "/fea81b1a-a77c-4c77-bfcb-f010ab6c4763" (reference "U3") (unit 1)))
+			(project "esp32_baseboard" (path "/b769966a-c1a5-4e09-8b47-a27c2881840e" (reference "U3") (unit 1)))
 		)
 	)
@@
 		(pin "4")
 		(instances
-			(project "esp32_baseboard" (path "/fea81b1a-a77c-4c77-bfcb-f010ab6c4763" (reference "J2") (unit 1)))
-		)
-	)
-	(symbol (lib_id "ESP32_Carrier:Conn_1x11_TFT") (at 215.9 139.7 0) (unit 1)
+			(project "esp32_baseboard" (path "/b769966a-c1a5-4e09-8b47-a27c2881840e" (reference "J2") (unit 1)))
+		)
+	)
+	(symbol (lib_id "ESP32_Carrier:Conn_1x10_TFT") (at 215.9 139.7 0) (unit 1)
 		(property "Reference" "J17" (at 215.9 126.99999999999999 0)
 			(effects (font (size 1.27 1.27)))
@@
 			(effects (font (size 1.27 1.27)))
 		)
-		(property "Footprint" "ESP32_Carrier:PinHeader_1x11_TFT" (at 215.9 139.7 0)
+		(property "Footprint" "ESP32_Carrier:PinHeader_1x10_TFT" (at 215.9 139.7 0)
 			(effects (font (size 1.27 1.27)) (hide yes))
 		)
@@
 		(pin "9")
 		(pin "10")
-		(pin "11")
-		(instances
-			(project "esp32_baseboard" (path "/fea81b1a-a77c-4c77-bfcb-f010ab6c4763" (reference "J17") (unit 1)))
+		(instances
+			(project "esp32_baseboard" (path "/b769966a-c1a5-4e09-8b47-a27c2881840e" (reference "J17") (unit 1)))
+		)
+	)
+	(symbol (lib_id "ESP32_Carrier:Conn_1x04_ENC") (at 265.0 139.7 0) (unit 1)
+		(property "Reference" "J18" (at 265.0 129.54 0)
+			(effects (font (size 1.27 1.27)))
+		)
+		(property "Value" "EC11_ENC" (at 265.0 149.85999999999999 0)
+			(effects (font (size 1.27 1.27)))
+		)
+		(property "Footprint" "ESP32_Carrier:PinHeader_1x04_ENC" (at 265.0 139.7 0)
+			(effects (font (size 1.27 1.27)) (hide yes))
+		)
+		(property "Datasheet" "~" (at 265.0 139.7 0)
+			(effects (font (size 1.27 1.27)) (hide yes))
+		)
+		(pin "1")
+		(pin "2")
+		(pin "3")
+		(pin "4")
+		(instances
+			(project "esp32_baseboard" (path "/b769966a-c1a5-4e09-8b47-a27c2881840e" (reference "J18") (unit 1)))
 		)
 	)
@@
 		(pin "12")
 		(instances
-			(project "esp32_baseboard" (path "/fea81b1a-a77c-4c77-bfcb-f010ab6c4763" (reference "U4") (unit 1)))
+			(project "esp32_baseboard" (path "/b769966a-c1a5-4e09-8b47-a27c2881840e" (reference "U4") (unit 1)))
 		)
 	)
@@
 		(pin "12")
 		(instances
-			(project "esp32_baseboard" (path "/fea81b1a-a77c-4c77-bfcb-f010ab6c4763" (reference "U9") (unit 1)))
+			(project "esp32_baseboard" (path "/b769966a-c1a5-4e09-8b47-a27c2881840e" (reference "U9") (unit 1)))
 		)
 	)
@@
 		(pin "10")
 		(instances
-			(project "esp32_baseboard" (path "/fea81b1a-a77c-4c77-bfcb-f010ab6c4763" (reference "J4") (unit 1)))
+			(project "esp32_baseboard" (path "/b769966a-c1a5-4e09-8b47-a27c2881840e" (reference "J4") (unit 1)))
 		)
 	)
@@
 		(effects (font (size 1.27 1.27)) (justify left bottom))
 	)
-	(wire
-		(pts (xy 305.24 93.98) (xy 324.32 93.98))
-		(stroke (width 0) (type default))
-	)
-	(wire
-		(pts (xy 324.32 93.98) (xy 324.32 97.79))
-		(stroke (width 0) (type default))
-	)
-	(wire
-		(pts (xy 324.32 97.79) (xy 147.32 97.79))
-		(stroke (width 0) (type default))
-	)
-	(label "OPTO_OUT8"
-		(at 324.32 93.98 0)
-		(effects (font (size 1.27 1.27)) (justify left bottom))
+	(text "J18 ENC: wall-mount EC11 cable → GND/3V3/A/B; CLK=IO9 DT=IO41; no SW"
+		(at 250.0 118.0 0)
+		(effects (font (size 1.0 1.0)) (justify left))
+	)
+	(wire
+		(pts (xy 147.32 97.79) (xy 257.0 97.79))
+		(stroke (width 0) (type default))
+	)
+	(wire
+		(pts (xy 257.0 97.79) (xy 265.0 140.97))
+		(stroke (width 0) (type default))
+	)
+	(label "ENC_A"
+		(at 259.0 140.97 0)
+		(effects (font (size 1.27 1.27)) (justify left bottom))
+	)
+	(wire
+		(pts (xy 182.88 77.47) (xy 259.0 77.47))
+		(stroke (width 0) (type default))
+	)
+	(wire
+		(pts (xy 259.0 77.47) (xy 265.0 143.51))
+		(stroke (width 0) (type default))
+	)
+	(label "ENC_B"
+		(at 259.0 143.51 0)
+		(effects (font (size 1.27 1.27)) (justify left bottom))
+	)
+	(wire
+		(pts (xy 265.0 135.89) (xy 255.0 135.89))
+		(stroke (width 0) (type default))
+	)
+	(wire
+		(pts (xy 255.0 135.89) (xy 255.0 73.66))
+		(stroke (width 0) (type default))
+	)
+	(wire
+		(pts (xy 255.0 73.66) (xy 147.32 73.66))
+		(stroke (width 0) (type default))
+	)
+	(wire
+		(pts (xy 265.0 138.43) (xy 253.0 138.43))
+		(stroke (width 0) (type default))
+	)
+	(wire
+		(pts (xy 253.0 138.43) (xy 253.0 35.56))
+		(stroke (width 0) (type default))
+	)
+	(wire
+		(pts (xy 253.0 35.56) (xy 147.32 35.56))
+		(stroke (width 0) (type default))
 	)
 	(text "BOTTOM: U5/U6/U7 DRV8871 @12V | TOP: J5/J6/J7 GA12-N20"
@@
 		(pin "6")
 		(instances
-			(project "esp32_baseboard" (path "/fea81b1a-a77c-4c77-bfcb-f010ab6c4763" (reference "U5") (unit 1)))
+			(project "esp32_baseboard" (path "/b769966a-c1a5-4e09-8b47-a27c2881840e" (reference "U5") (unit 1)))
 		)
 	)
@@
 		(pin "2")
 		(instances
-			(project "esp32_baseboard" (path "/fea81b1a-a77c-4c77-bfcb-f010ab6c4763" (reference "J5") (unit 1)))
+			(project "esp32_baseboard" (path "/b769966a-c1a5-4e09-8b47-a27c2881840e" (reference "J5") (unit 1)))
 		)
 	)
@@
 		(pin "2")
 		(instances
-			(project "esp32_baseboard" (path "/fea81b1a-a77c-4c77-bfcb-f010ab6c4763" (reference "J8") (unit 1)))
+			(project "esp32_baseboard" (path "/b769966a-c1a5-4e09-8b47-a27c2881840e" (reference "J8") (unit 1)))
 		)
 	)
@@
 		(pin "2")
 		(instances
-			(project "esp32_baseboard" (path "/fea81b1a-a77c-4c77-bfcb-f010ab6c4763" (reference "J9") (unit 1)))
+			(project "esp32_baseboard" (path "/b769966a-c1a5-4e09-8b47-a27c2881840e" (reference "J9") (unit 1)))
 		)
 	)
@@
 		(pin "6")
 		(instances
-			(project "esp32_baseboard" (path "/fea81b1a-a77c-4c77-bfcb-f010ab6c4763" (reference "U6") (unit 1)))
+			(project "esp32_baseboard" (path "/b769966a-c1a5-4e09-8b47-a27c2881840e" (reference "U6") (unit 1)))
 		)
 	)
@@
 		(pin "2")
 		(instances
-			(project "esp32_baseboard" (path "/fea81b1a-a77c-4c77-bfcb-f010ab6c4763" (reference "J6") (unit 1)))
+			(project "esp32_baseboard" (path "/b769966a-c1a5-4e09-8b47-a27c2881840e" (reference "J6") (unit 1)))
 		)
 	)
@@
 		(pin "2")
 		(instances
-			(project "esp32_baseboard" (path "/fea81b1a-a77c-4c77-bfcb-f010ab6c4763" (reference "J10") (unit 1)))
+			(project "esp32_baseboard" (path "/b769966a-c1a5-4e09-8b47-a27c2881840e" (reference "J10") (unit 1)))
 		)
 	)
@@
 		(pin "2")
 		(instances
-			(project "esp32_baseboard" (path "/fea81b1a-a77c-4c77-bfcb-f010ab6c4763" (reference "J11") (unit 1)))
+			(project "esp32_baseboard" (path "/b769966a-c1a5-4e09-8b47-a27c2881840e" (reference "J11") (unit 1)))
 		)
 	)
@@
 		(pin "6")
 		(instances
-			(project "esp32_baseboard" (path "/fea81b1a-a77c-4c77-bfcb-f010ab6c4763" (reference "U7") (unit 1)))
+			(project "esp32_baseboard" (path "/b769966a-c1a5-4e09-8b47-a27c2881840e" (reference "U7") (unit 1)))
 		)
 	)
@@
 		(pin "2")
 		(instances
-			(project "esp32_baseboard" (path "/fea81b1a-a77c-4c77-bfcb-f010ab6c4763" (reference "J7") (unit 1)))
+			(project "esp32_baseboard" (path "/b769966a-c1a5-4e09-8b47-a27c2881840e" (reference "J7") (unit 1)))
 		)
 	)
@@
 		(pin "2")
 		(instances
-			(project "esp32_baseboard" (path "/fea81b1a-a77c-4c77-bfcb-f010ab6c4763" (reference "J12") (unit 1)))
+			(project "esp32_baseboard" (path "/b769966a-c1a5-4e09-8b47-a27c2881840e" (reference "J12") (unit 1)))
 		)
 	)
@@
 		(pin "2")
 		(instances
-			(project "esp32_baseboard" (path "/fea81b1a-a77c-4c77-bfcb-f010ab6c4763" (reference "J13") (unit 1)))
+			(project "esp32_baseboard" (path "/b769966a-c1a5-4e09-8b47-a27c2881840e" (reference "J13") (unit 1)))
 		)
 	)
@@
 		(pin "4")
 		(instances
-			(project "esp32_baseboard" (path "/fea81b1a-a77c-4c77-bfcb-f010ab6c4763" (reference "J14") (unit 1)))
+			(project "esp32_baseboard" (path "/b769966a-c1a5-4e09-8b47-a27c2881840e" (reference "J14") (unit 1)))
 		)
 	)
@@
 		(pin "2")
 		(instances
-			(project "esp32_baseboard" (path "/fea81b1a-a77c-4c77-bfcb-f010ab6c4763" (reference "R1") (unit 1)))
+			(project "esp32_baseboard" (path "/b769966a-c1a5-4e09-8b47-a27c2881840e" (reference "R1") (unit 1)))
 		)
 	)
@@
 		(pin "1")
 		(instances
-			(project "esp32_baseboard" (path "/fea81b1a-a77c-4c77-bfcb-f010ab6c4763" (reference "#FLG1") (unit 1)))
-		)
-	)
+			(project "esp32_baseboard" (path "/b769966a-c1a5-4e09-8b47-a27c2881840e" (reference "#FLG1") (unit 1)))
+		)
+	)

Commit message: tmp
Parts:
- added C10: 47u/25V, ESP32_Carrier:CP_Radial_D6_47u_25V, symbol ESP32_Carrier:GEN_CP_Radial_D6_47u_25V
- added C11: 100n, ESP32_Carrier:C_0805_100n, symbol ESP32_Carrier:GEN_C_0805_100n
- added C20, C21, C22, C23: 470u/25V, ESP32_Carrier:CP_Radial_D8_470u_25V, symbol ESP32_Carrier:GEN_CP_Radial_D8_470u_25V
- added D1: P6KE15A, ESP32_Carrier:Diode_TVS_DO41, symbol ESP32_Carrier:GEN_Diode_TVS_DO41
- added D2: 1N5819, ESP32_Carrier:Diode_TVS_DO41, symbol ESP32_Carrier:GEN_Diode_TVS_DO41
- added F1: PTC_3A_30V, ESP32_Carrier:Fuse_PTC_Radial_5.1mm, symbol ESP32_Carrier:GEN_Fuse_PTC_Radial_5_1mm
- added J15: BUZZER_5V, ESP32_Carrier:PinHeader_1x03_Buzzer, symbol ESP32_Carrier:GEN_PinHeader_1x03_Buzzer
- added J16: AOD4184, ESP32_Carrier:PinHeader_1x04_MOSFET, symbol ESP32_Carrier:GEN_PinHeader_1x04_MOSFET
- added R10: 10R, ESP32_Carrier:R_1206_10R, symbol ESP32_Carrier:GEN_R_1206_10R
- added R2, R3: 10k, ESP32_Carrier:R_Axial_4k7_BUP, symbol ESP32_Carrier:R_BUP_Pullup
- U3: value TMC2209_StepStick -> TMC2209
Connections:
- net +12V: now also C20.1 (P1), C21.1 (P1), C22.1 (P1), C23.1 (P1), D1.2 (P2), D2.1 (P1), F1.2 (P2), J16.3 (P3), R10.1 (P1); no longer J1.1 (+12V), J1.2 (GND), J14.2 (GND), J18.1 (GND), J18.2 (3V3), J4.1 (GND_I), J4.2 (VCC_I), U1.1 (3V3), U1.21 (5V), U1.22 (GND), U2.2 (VIN-), U2.3 (VOUT+), U2.4 (VOUT-), U3.10 (GND), U3.15 (VIO), U3.16 (GND2), U4.1 (GND_I), U4.2 (VCC_I), U4.7 (GND_O), U4.8 (VCC_O), U5.2 (GND), U6.2 (GND), U7.2 (GND), U9.1 (GND_I), U9.2 (VCC_I), U9.7 (GND_O), U9.8 (VCC_O)
- net +12V_SNS: now also C10.1 (P1), C11.1 (P1), R10.2 (P2)
- net ENC_A: now also J18.3 (ENC_A), U1.32 (IO38)
- net ENC_B: now also J18.4 (ENC_B), U1.29 (IO41)
- net OPTO_IN5: now also J4.7 (IN5), U9.3 (IN1)
- net OPTO_IN6: now also J4.8 (IN6), U9.4 (IN2)
- net OPTO_IN7: now also J4.9 (IN7), U9.5 (IN3)
- net OPTO_IN8: now also J4.10 (IN8), U9.6 (IN4)
- net OPTO_OUT1: no longer U1.4 (IO4), U4.11 (OUT3)
- net OPTO_OUT2: no longer U1.5 (IO5), U4.12 (OUT4)
- net OPTO_OUT6: no longer J18.4 (ENC_B), U1.29 (IO41)
- net STEP: no longer J2.4 (B2), U3.14 (B2)
- net GND: now reaches J17.1 (GND)
- net GND: now also J1.2 (GND), J14.2 (GND), J18.1 (GND), J4.1 (GND_I), U1.22 (GND), U1.23 (GND), U1.43 (GNDb), U1.44 (GNDc), U2.2 (VIN-), U2.4 (VOUT-), U3.10 (GND), U3.16 (GND2), U4.1 (GND_I), U4.7 (GND_O), U5.2 (GND), U6.2 (GND), U7.2 (GND), U9.1 (GND_I), U9.7 (GND_O), C10.2 (P2), C11.2 (P2), C20.2 (P2), C21.2 (P2), C22.2 (P2), C23.2 (P2), D1.1 (P1), J15.2 (P2), J16.2 (P2), R3.2
- net T_CS: now reaches J17.10 (T_CS)
- net T_CS: now also U1.38 (IO48)
- net +3V3: now reaches J17.2 (3V3)
- net +3V3: now also J18.2 (3V3), U1.1 (3V3), U1.2 (3V3b), U3.15 (VIO), U4.8 (VCC_O), U9.8 (VCC_O), R2.2
- net TFT_SCK: now reaches J17.3 (SCK)
- net TFT_SCK: now also U1.31 (IO39)
- net TFT_MOSI: now reaches J17.4 (MOSI)
- net TFT_MOSI: now also U1.30 (IO40)
- net TFT_MISO: now reaches J17.5 (MISO)
- net TFT_MISO: now also U1.39 (IO47)
- net TFT_CS: now reaches J17.6 (CS)
- net TFT_CS: now also U1.28 (IO42)
- net TFT_DC: now reaches J17.7 (DC)
- net TFT_DC: now also U1.40 (IO21)
- net TFT_RST: now reaches J17.8 (RST)
- net TFT_RST: now also U1.14 (IO46)
- net TFT_BL: now reaches J17.9 (BL)
- net TFT_BL: now also U1.37 (IO45)
- net MotDC1_A: now reaches J5.1 (M+), U5.5 (OUT1)
- net MotDC1_B: now reaches J5.2 (M-), U5.6 (OUT2)
- net MotA2: now reaches J2.1 (A2), U3.11 (A2)
- net MotA1: now reaches J2.2 (A1), U3.12 (A1)
- net OPTO_OUT8: now reaches U9.12 (OUT4)
- net MotDC3_A: now reaches J7.1 (M+), U7.5 (OUT1)
- net MotDC3_B: now reaches J7.2 (M-), U7.6 (OUT2)
- net BLOWER: now reaches U1.13 (IO3)
- net BLOWER: now also J16.1 (P1), R3.1
- net BUZZER: now reaches U1.15 (IO9)
- net BUZZER: now also J15.3 (P3); no longer J18.3 (ENC_A)
- net MotDC2_A: now reaches J6.1 (M+), U6.5 (OUT1)
- net MotDC2_B: now reaches J6.2 (M-), U6.6 (OUT2)
- net EN renamed EN_TMC
- net EN_TMC: now also R2.1; no longer J2.3 (B1), U3.13 (B1)
- net U5_IN1 renamed DC1_IN1
- net U5_IN2 renamed DC1_IN2
- net U6_IN1 renamed DC2_IN1
- net U6_IN2 renamed DC2_IN2
- net U7_IN1 renamed DC3_IN1
- net U7_IN2 renamed DC3_IN2
- new net +12V_RAW: F1.1 (P1), J1.1 (+12V)
- new net +5V: J15.1 (P1), U1.21 (5V), U2.3 (VOUT+)
- new net BLW_RET: D2.2 (P2), J16.4 (P4)
- new net MotB1: J2.3 (B1), U3.13 (B1)
- new net MotB2: J2.4 (B2), U3.14 (B2)
- new net OPTO_OUT3: U1.4 (IO4), U4.11 (OUT3)
- new net OPTO_OUT4: U1.5 (IO5), U4.12 (OUT4)
- new net OPTO_VCC_I: J4.2 (VCC_I), U4.2 (VCC_I), U9.2 (VCC_I)
- no-connect marks 6 -> 15
Other:
- note removed: "BOTTOM: J1 12V + MP1584EN + TMC2209 + ESP32"
- note removed: "BOTTOM: U5/U6/U7 DRV8871 @12V | TOP: J5/J6/J7 GA12-N20"
- note removed: "BUP-30S NPN: Nau=+12 Xanh=GND Den=OUT Trang=CTRL"
- note removed: "Bulk 470u tai moi DRV8871/TMC (tren PCB)"
- note removed: "CTRL: LightON->+12V / DarkON->GND"
- note removed: "GND_I=GND (limit SW @12V shared)"
- note removed: "J18 ENC: wall-mount EC11 cable → GND/3V3/A/B; CLK=IO9 DT=IO41; no SW"
- note removed: "R10 10R + C10 47u + C11 100n (tren PCB)"
- note removed: "STAR: +12V_MOT (rong) / +12V_SNS qua R10=10R + C47u||100n"
- note removed: "TOP: J2 NEMA17 / J17 TFT / J18 ENC / J15 buzzer / J16 MOSFET"
- note removed: "TRUC1 MOT+LIM"
- note removed: "TRUC2 MOT+LIM"
- note removed: "TRUC3 MOT+LIM"
- note removed: "U4+U9 PC817 4ch x2 + J4 field IN (TOP)"
- title: ESP32-S3 Baseboard - MP1584 + TMC + Opto + 3x DRV8871 -> (none)

Commit message: sắp xếp và chọn lại linh kiện cho PCB
Parts:
- removed C10: 47u/25V, ESP32_Carrier:CP_Radial_D6_47u_25V, symbol ESP32_Carrier:GEN_CP_Radial_D6_47u_25V
- removed C11: 100n, ESP32_Carrier:C_0805_100n, symbol ESP32_Carrier:GEN_C_0805_100n
- removed C20, C21, C22, C23: 470u/25V, ESP32_Carrier:CP_Radial_D8_470u_25V, symbol ESP32_Carrier:GEN_CP_Radial_D8_470u_25V
- removed D1: P6KE15A, ESP32_Carrier:Diode_TVS_DO41, symbol ESP32_Carrier:GEN_Diode_TVS_DO41
- removed D2: 1N5819, ESP32_Carrier:Diode_TVS_DO41, symbol ESP32_Carrier:GEN_Diode_TVS_DO41
- removed F1: PTC_3A_30V, ESP32_Carrier:Fuse_PTC_Radial_5.1mm, symbol ESP32_Carrier:GEN_Fuse_PTC_Radial_5_1mm
- removed J10, J12, J8: LIM_MIN_NC, ESP32_Carrier:PinHeader_1x02_LimitSW, symbol ESP32_Carrier:Conn_1x02_LimitSW
- removed J11, J13, J9: LIM_MAX_NC, ESP32_Carrier:PinHeader_1x02_LimitSW, symbol ESP32_Carrier:Conn_1x02_LimitSW
- removed J15: BUZZER_5V, ESP32_Carrier:PinHeader_1x03_Buzzer, symbol ESP32_Carrier:GEN_PinHeader_1x03_Buzzer
- removed J16: AOD4184, ESP32_Carrier:PinHeader_1x04_MOSFET, symbol ESP32_Carrier:GEN_PinHeader_1x04_MOSFET
- removed J17: TFT_TOUCH, ESP32_Carrier:PinHeader_1x10_TFT, symbol ESP32_Carrier:Conn_1x10_TFT
- removed J4: OPTO_FIELD_IN, ESP32_Carrier:PinHeader_1x10_OptoField, symbol ESP32_Carrier:Conn_1x10_OptoField
- removed J5, J6, J7: GA12_N20, ESP32_Carrier:PinHeader_1x02_MotorDC, symbol ESP32_Carrier:Conn_1x02_MotorDC
- removed R10: 10R, ESP32_Carrier:R_1206_10R, symbol ESP32_Carrier:GEN_R_1206_10R
- removed R2, R3: 10k, ESP32_Carrier:R_Axial_4k7_BUP, symbol ESP32_Carrier:R_BUP_Pullup
- removed U4, U9: PC817_4CH, ESP32_Carrier:PC817_4CH_Opto, symbol ESP32_Carrier:PC817_4CH_Opto
- removed U5, U6, U7: DRV8871_Module, ESP32_Carrier:DRV8871_Module, symbol ESP32_Carrier:DRV8871_Module
- added J10: END_HOME2, ESP32_Carrier:PinHeader_1x04_Endstop, symbol ESP32_Carrier:Conn_1x04_Endstop
- added J12: END_HOME3, ESP32_Carrier:PinHeader_1x04_Endstop, symbol ESP32_Carrier:Conn_1x04_Endstop
- added J17: TFT_LCD_1x09, ESP32_Carrier:PinHeader_1x09_TFT_LCD, symbol ESP32_Carrier:Conn_1x09_TFT_LCD
- added J23: TFT_TP_1x05, ESP32_Carrier:PinHeader_1x05_TFT_TP, symbol ESP32_Carrier:Conn_1x05_TFT_TP
- added J8: END_HOME1, ESP32_Carrier:PinHeader_1x04_Endstop, symbol ESP32_Carrier:Conn_1x04_Endstop
- added U41, U42, U43, U44: PC817, ESP32_Carrier:PC817_DIP4, symbol ESP32_Carrier:PC817_DIP4
- U3: value TMC2209 -> TMC2209_StepStick
Connections:
- net +12V_RAW is gone; now on net +12V: J1.1 (+12V)
- net +5V is gone; now on net +12V: U1.21 (5V), U2.3 (VOUT+)
- net MotB1 is gone; now on net /EN: J2.3 (B1), U3.13 (B1)
- net STEP is gone; now on net /STEP: U1.9 (IO16), U3.7 (STEP)
- net +12V: now also J1.2 (GND), J14.2 (GND), J18.1 (GND), J18.2 (3V3), U1.1 (3V3), U1.22 (GND), U2.2 (VIN-), U2.4 (VOUT-), U3.10 (GND), U3.15 (VIO), U3.16 (GND2)
- net +12V_SNS: now also J10.3 (SIG), J10.4 (SNS), J12.3 (SIG), J12.4 (SNS), J8.3 (SIG), J8.4 (SNS)
- removed net +3V3: J18.2 (3V3), U1.1 (3V3), U1.2 (3V3b), U3.15 (VIO)
- net BLOWER: no longer names the net of U1.13 (IO3)
- net BUZZER: no longer names the net of U1.15 (IO9)
- net DC1_IN1: no longer names the net of U1.16 (IO10)
- net DC1_IN2: no longer names the net of U1.17 (IO11)
- net DC2_IN1: no longer names the net of U1.18 (IO12)
- net DC2_IN2: no longer names the net of U1.19 (IO13)
- net DC3_IN1: no longer names the net of U1.20 (IO14)
- net DC3_IN2: no longer names the net of U1.8 (IO15)
- net DIR renamed /DIR
- net ENC_A: no longer names the net of J18.3 (ENC_A), U1.32 (IO38)
- net ENC_B: no longer names the net of J18.4 (ENC_B), U1.29 (IO41)
- net EN_TMC renamed /EN
- removed net GND: J1.2 (GND), J14.2 (GND), J18.1 (GND), U1.22 (GND), U1.23 (GND), U1.43 (GNDb), U1.44 (GNDc), U2.2 (VIN-), U2.4 (VOUT-), U3.10 (GND), U3.16 (GND2)
- net MotA1: no longer names the net of J2.2 (A1), U3.12 (A1)
- net MotA2: no longer names the net of J2.1 (A2), U3.11 (A2)
- net MotB2 renamed /STEP
- net OPTO_IN7 renamed /OPTO_IN4
- net OPTO_OUT1: no longer names the net of U1.26 (IO1)
- net OPTO_OUT2: no longer names the net of U1.27 (IO2)
- net OPTO_OUT3: no longer names the net of U1.4 (IO4)
- net OPTO_OUT4: no longer names the net of U1.5 (IO5)
- net OPTO_OUT5: no longer names the net of U1.6 (IO6)
- net OPTO_OUT6: no longer names the net of U1.7 (IO7)
- net OPTO_OUT7: no longer names the net of U1.12 (IO8)
- net TFT_BL: no longer names the net of U1.37 (IO45)
- net TFT_CS: no longer names the net of U1.28 (IO42)
- net TFT_DC: no longer names the net of U1.40 (IO21)
- net TFT_MISO: no longer names the net of U1.39 (IO47)
- net TFT_MOSI: no longer names the net of U1.30 (IO40)
- net TFT_RST: no longer names the net of U1.14 (IO46)
- net TFT_SCK: no longer names the net of U1.31 (IO39)
- net T_CS: no longer names the net of U1.38 (IO48)
- no-connect marks 15 -> 6
Other:
- note added: "1_Q0-3->U5; 1_Q4-7->U6; 2_Q0-3->U7; shift 3 bytes; COM=+12V"
- note added: "BOTTOM: J1 12V + MP1584EN + TMC2209 + ESP32"
- note added: "BUP"
- note added: "BUP-30S NPN -> OPTO_IN4 (was IN7)"
- note added: "Bulk C20 470u@TMC + C21 100u shared ULN COM (tren PCB)"
- note added: "CTRL LDEN/GND/VCC/LDSI/LDSTR/LDSCK = OE/GND/3V3/SER/RCLK/SRCLK; R4 LDEN PU"
- note added: "CTRL: LightON->+12V / DarkON->GND"
- note added: "HOME1"
- note added: "HOME2"
- note added: "HOME3"
- note added: "IN: HOME×3 + BUP only (no field)"
- note added: "J18 ENC: wall-mount EC11 → GND/3V3/A/B; CLK=IO38 DT=IO41; no SW"
- note added: "R10 10R + C10 47u + C11 100n (tren PCB)"
- note added: "STAR: +12V_MOT (rong) / +12V_SNS qua R10=10R + C47u||100n"
- note added: "TOP: J17+J23 TFT / J18 ENC / J15 buzzer / J16 MOSFET"
- note added: "U10=74HC595-24IO module (Shopee) RIGHT of ESP32; U5-U7 ULN; J5-J7 BYJ"
- note added: "U41-U44 PC817 DIP-4 + 2k2/10k (HOME×3+BUP)"
- title: (none) -> ESP32-S3 Baseboard - MP1584 + TMC + ULN2003 direct GPIO
