File: pcb/esp32_baseboard/esp32_baseboard.kicad_sch (KiCad schematic)
At the start: 17 parts, among them J1 Screw_12V_IN, J10 END_HOME2, J12 END_HOME3, J14 BUP_30S, J17 TFT_LCD_1x09, J18 EC11_ENC, J2 NEMA17_OUT, J23 TFT_TP_1x05, J8 END_HOME1, U1 ESP32_S3_DevKitC_1, U2 MP1584_5V3A, U3 TMC2209_StepStick, U41 PC817, U42 PC817, U43 PC817, U44 PC817

Commit message: đi dây cho mạch PCB
Parts:
- removed J2: NEMA17_OUT, ESP32_Carrier:PinHeader_1x04_Motor, symbol ESP32_Carrier:Conn_1x04_Motor
- added C10: 47u/25V, ESP32_Carrier:CP_Radial_D6_47u_25V, symbol ESP32_Carrier:GEN_CP_Radial_D6_47u_25V
- added C11: 100n, ESP32_Carrier:C_0805_100n, symbol ESP32_Carrier:GEN_C_0805_100n
- added C20: 470u/25V, ESP32_Carrier:CP_Radial_D8_470u_25V, symbol ESP32_Carrier:GEN_CP_Radial_D8_470u_25V
- added C21: 100u/25V, ESP32_Carrier:CP_Radial_D6_100u_25V, symbol ESP32_Carrier:GEN_CP_Radial_D6_100u_25V
- added D1: P6KE15A, ESP32_Carrier:Diode_TVS_DO41, symbol ESP32_Carrier:GEN_Diode_TVS_DO41
- added D2: 1N5819, ESP32_Carrier:Diode_TVS_DO41, symbol ESP32_Carrier:GEN_Diode_TVS_DO41
- added F1: PTC_3A_30V, ESP32_Carrier:Fuse_PTC_Radial_5.1mm, symbol ESP32_Carrier:GEN_Fuse_PTC_Radial_5_1mm
- added J15: BUZZER_5V, ESP32_Carrier:PinHeader_1x03_Buzzer, symbol ESP32_Carrier:GEN_PinHeader_1x03_Buzzer
- added J16: AOD4184, ESP32_Carrier:PinHeader_1x04_MOSFET, symbol ESP32_Carrier:GEN_PinHeader_1x04_MOSFET
- added J24: 595_CTRL, ESP32_Carrier:PinHeader_1x06_595CTRL, symbol ESP32_Carrier:GEN_PinHeader_1x06_595CTRL
- added J25: 595_Q, ESP32_Carrier:PinHeader_1x24_595Q, symbol ESP32_Carrier:GEN_PinHeader_1x24_595Q
- added J5, J6, J7: 28BYJ48, ESP32_Carrier:PinHeader_1x05_BYJ, symbol ESP32_Carrier:Conn_1x05_BYJ
- added R10: 10R, ESP32_Carrier:R_1206_10R, symbol ESP32_Carrier:GEN_R_1206_10R
- added R2, R3, R4, R45, R46, R47, R48: 10k, ESP32_Carrier:R_Axial_4k7_BUP, symbol ESP32_Carrier:R_BUP_Pullup
- added R41, R42, R43, R44: 2k2, ESP32_Carrier:R_Axial_4k7_BUP, symbol ESP32_Carrier:R_BUP_Pullup
- added U5, U6, U7: ULN2003AN, ESP32_Carrier:ULN2003AN, symbol ESP32_Carrier:ULN2003AN
- J17: value TFT_LCD_1x09 -> TFT_LCD
- J23: value TFT_TP_1x05 -> TFT_TP
- U3: value TMC2209_StepStick -> TMC2209
Connections:
- net +12V: now also C20.1 (P1), C21.1 (P1), D1.2 (P2), D2.1 (P1), F1.2 (P2), J16.3 (P3), J5.5 (+12V), J6.5 (+12V), J7.5 (+12V), R10.1 (P1), U5.9 (COM), U6.9 (COM), U7.9 (COM); no longer J1.1 (+12V), J1.2 (GND), J14.2 (GND), J18.1 (GND), J18.2 (3V3), U1.1 (3V3), U1.21 (5V), U1.22 (GND), U2.2 (VIN-), U2.3 (VOUT+), U2.4 (VOUT-), U3.10 (GND), U3.15 (VIO), U3.16 (GND2)
- net +12V_SNS: now also C10.1 (P1), C11.1 (P1), R10.2 (P2); no longer J10.3 (SIG), J12.3 (SIG), J8.3 (SIG)
- net OPTO_A3: now reaches U43.1 (A)
- net OPTO_A3: now also R43.2
- net GND: now reaches U43.2 (K)
- net GND: now also J1.2 (GND), J14.2 (GND), J17.2 (GND), J18.1 (GND), U1.22 (GND), U1.23 (GND), U1.43 (GNDb), U1.44 (GNDc), U2.2 (VIN-), U2.3 (VOUT+), U3.10 (GND), U3.16 (GND2), U41.2 (K), U41.3 (E), U42.2 (K), U42.3 (E), U43.3 (E), U44.2 (K), U44.3 (E), C10.2 (P2), C11.2 (P2), C20.2 (P2), C21.2 (P2), D1.1 (P1), J15.2 (P2), J16.2 (P2), J24.2 (P2), R3.2, U5.8 (GND), U6.8 (GND), U7.8 (GND)
- net OPTO_OUT3: now reaches U43.4 (C)
- net OPTO_OUT3: now also U1.4 (IO4), R47.2
- net TFT_SCK: now reaches J23.1 (T_CLK)
- net TFT_SCK: now also J17.7 (SCK), U1.31 (IO39)
- net T_CS: now reaches J23.2 (T_CS)
- net T_CS: now also U1.38 (IO48)
- net TFT_MOSI: now reaches J23.3 (T_DIN)
- net TFT_MOSI: now also J17.6 (SDI), U1.30 (IO40)
- net TFT_MISO: now reaches J23.4 (T_DO)
- net TFT_MISO: now also U1.39 (IO47)
- net T_IRQ: now reaches J23.5 (T_IRQ)
- net T_IRQ: now also U1.6 (IO6)
- net MotA2: now reaches U3.11 (A2)
- net MotA1: now reaches U3.12 (A1)
- net OPTO_A4: now reaches U44.1 (A)
- net OPTO_A4: now also R44.2
- net OPTO_OUT4: now reaches U44.4 (C)
- net OPTO_OUT4: now also U1.5 (IO5), R48.2
- net ENC_A: now reaches J18.3 (ENC_A), U1.32 (IO38)
- net ENC_B: now reaches J18.4 (ENC_B), U1.29 (IO41)
- net OPTO_A2: now reaches U42.1 (A)
- net OPTO_A2: now also R42.2
- net OPTO_OUT2: now reaches U42.4 (C)
- net OPTO_OUT2: now also U1.27 (IO2), R46.2
- net +3V3: now reaches J17.1 (VCC)
- net +3V3: now also J18.2 (3V3), U1.1 (3V3), U1.2 (3V3b), U3.15 (VIO), J24.3 (P3), R2.2, R4.2, R45.1, R46.1, R47.1, R48.1
- net TFT_CS: now reaches J17.3 (CS)
- net TFT_CS: now also U1.28 (IO42)
- net TFT_RST: now reaches J17.4 (RESET)
- net TFT_RST: now also U1.14 (IO46)
- net TFT_DC: now reaches J17.5 (DC)
- net TFT_DC: now also U1.40 (IO21)
- net TFT_BL: now reaches J17.8 (LED)
- net TFT_BL: now also U1.37 (IO45)
- net OPTO_A1: now reaches U41.1 (A)
- net OPTO_A1: now also R41.2
- net OPTO_OUT1: now reaches U41.4 (C)
- net OPTO_OUT1: now also U1.26 (IO1), R45.2
- net BLOWER: now reaches U1.13 (IO3)
- net BLOWER: now also J16.1 (P1), R3.1
- net BUZZER: now reaches U1.15 (IO9)
- net BUZZER: now also J15.3 (P3)
- net SER: now reaches U1.16 (IO10)
- net SER: now also J24.4 (P4)
- net SRCLK: now reaches U1.17 (IO11)
- net SRCLK: now also J24.6 (P6)
- net RCLK: now reaches U1.18 (IO12)
- net RCLK: now also J24.5 (P5)
- net OE_595: now reaches U1.19 (IO13)
- net OE_595: now also J24.1 (P1), R4.1
- net /DIR renamed DIR
- net /EN renamed EN_TMC
- net EN_TMC: now also R2.1; no longer U3.13 (B1)
- net /OPTO_IN4 renamed OPTO_IN4
- net OPTO_IN4: now also R44.1
- net /STEP renamed STEP
- net STEP: no longer U3.14 (B2)
- new net +12V_RAW: F1.1 (P1), J1.1 (+12V)
- new net +5V: J15.1 (P1), U1.21 (5V), U2.4 (VOUT-)
- new net BLW_RET: D2.2 (P2), J16.4 (P4)
- new net BYJ1_A: J5.1 (A), U5.16 (OUT1)
- new net BYJ1_B: J5.2 (B), U5.15 (OUT2)
- new net BYJ1_C: J5.3 (C), U5.14 (OUT3)
- new net BYJ1_D: J5.4 (D), U5.13 (OUT4)
- new net BYJ2_A: J6.1 (A), U6.16 (OUT1)
- new net BYJ2_B: J6.2 (B), U6.15 (OUT2)
- new net BYJ2_C: J6.3 (C), U6.14 (OUT3)
- new net BYJ2_D: J6.4 (D), U6.13 (OUT4)
- new net BYJ3_A: J7.1 (A), U7.16 (OUT1)
- new net BYJ3_B: J7.2 (B), U7.15 (OUT2)
- new net BYJ3_C: J7.3 (C), U7.14 (OUT3)
- new net BYJ3_D: J7.4 (D), U7.13 (OUT4)
- new net MotB1: U3.13 (B1)
- new net MotB2: U3.14 (B2)
- new net OPTO_IN1: J8.3 (SIG), R41.1
- new net OPTO_IN2: J10.3 (SIG), R42.1
- new net OPTO_IN3: J12.3 (SIG), R43.1
- new net SR_Q0: J25.1 (P1), U5.1 (IN1)
- new net SR_Q1: J25.2 (P2), U5.2 (IN2)
- new net SR_Q10: J25.11 (P11), U7.3 (IN3)
- new net SR_Q11: J25.12 (P12), U7.4 (IN4)
- new net SR_Q2: J25.3 (P3), U5.3 (IN3)
- new net SR_Q3: J25.4 (P4), U5.4 (IN4)
- new net SR_Q4: J25.5 (P5), U6.1 (IN1)
- new net SR_Q5: J25.6 (P6), U6.2 (IN2)
- new net SR_Q6: J25.7 (P7), U6.3 (IN3)
- new net SR_Q7: J25.8 (P8), U6.4 (IN4)
- new net SR_Q8: J25.9 (P9), U7.1 (IN1)
- new net SR_Q9: J25.10 (P10), U7.2 (IN2)
- no-connect marks 6 -> 56
Other:
- note removed: "1_Q0-3->U5; 1_Q4-7->U6; 2_Q0-3->U7; shift 3 bytes; COM=+12V"
- note removed: "BOTTOM: J1 12V + MP1584EN + TMC2209 + ESP32"
- note removed: "BUP"
- note removed: "BUP-30S NPN -> OPTO_IN4 (was IN7)"
- note removed: "Bulk C20 470u@TMC + C21 100u shared ULN COM (tren PCB)"
- note removed: "CTRL LDEN/GND/VCC/LDSI/LDSTR/LDSCK = OE/GND/3V3/SER/RCLK/SRCLK; R4 LDEN PU"
- note removed: "CTRL: LightON->+12V / DarkON->GND"
- note removed: "HOME1"
- note removed: "HOME2"
- note removed: "HOME3"
- note removed: "IN: HOME×3 + BUP only (no field)"
- note removed: "J18 ENC: wall-mount EC11 → GND/3V3/A/B; CLK=IO38 DT=IO41; no SW"
- note removed: "R10 10R + C10 47u + C11 100n (tren PCB)"
- note removed: "STAR: +12V_MOT (rong) / +12V_SNS qua R10=10R + C47u||100n"
- note removed: "TOP: J17+J23 TFT / J18 ENC / J15 buzzer / J16 MOSFET"
- note removed: "U10=74HC595-24IO module (Shopee) RIGHT of ESP32; U5-U7 ULN; J5-J7 BYJ"
- note removed: "U41-U44 PC817 DIP-4 + 2k2/10k (HOME×3+BUP)"
- title: ESP32-S3 Baseboard - MP1584 + TMC + ULN2003 direct GPIO -> (none)

Commit message: update PCB cho phần power và opto và sắp xếp linh kiện
Parts:
- removed F1: PTC_3A_30V, ESP32_Carrier:Fuse_PTC_Radial_5.1mm, symbol ESP32_Carrier:GEN_Fuse_PTC_Radial_5_1mm
- removed J10: END_HOME2, ESP32_Carrier:PinHeader_1x04_Endstop, symbol ESP32_Carrier:Conn_1x04_Endstop
- removed J12: END_HOME3, ESP32_Carrier:PinHeader_1x04_Endstop, symbol ESP32_Carrier:Conn_1x04_Endstop
- removed J14: BUP_30S, ESP32_Carrier:PinHeader_1x04_BUP30S, symbol ESP32_Carrier:Conn_1x04_BUP30S
- removed J15: BUZZER_5V, ESP32_Carrier:PinHeader_1x03_Buzzer, symbol ESP32_Carrier:GEN_PinHeader_1x03_Buzzer
- removed J16: AOD4184, ESP32_Carrier:PinHeader_1x04_MOSFET, symbol ESP32_Carrier:GEN_PinHeader_1x04_MOSFET
- removed J18: EC11_ENC, ESP32_Carrier:PinHeader_1x04_ENC, symbol ESP32_Carrier:Conn_1x04_ENC
- removed J5, J6, J7: 28BYJ48, ESP32_Carrier:PinHeader_1x05_BYJ, symbol ESP32_Carrier:Conn_1x05_BYJ
- removed J8: END_HOME1, ESP32_Carrier:PinHeader_1x04_Endstop, symbol ESP32_Carrier:Conn_1x04_Endstop
- removed U5, U6, U7: ULN2003AN, ESP32_Carrier:ULN2003AN, symbol ESP32_Carrier:ULN2003AN
- added C24, C25: 100n, ESP32_Carrier:C_0805_100n, symbol ESP32_Carrier:GEN_C_0805_100n
- added C26: 100n SNS, ESP32_Carrier:C_0805_100n, symbol ESP32_Carrier:GEN_C_0805_100n
- added D3: SS54, ESP32_Carrier:Diode_TVS_DO41, symbol ESP32_Carrier:GEN_Diode_TVS_DO41
- added F1: 5x20 T3.15A, ESP32_Carrier:Fuse_Holder_5x20_Open, symbol ESP32_Carrier:GEN_Fuse_Holder_5x20_Open
- added J10: HOME HOME2, ESP32_Carrier:JST_XH_02_Socket, symbol ESP32_Carrier:Conn_JST_XH_02
- added J12: HOME HOME3, ESP32_Carrier:JST_XH_02_Socket, symbol ESP32_Carrier:Conn_JST_XH_02
- added J14: BUP-30S, ESP32_Carrier:JST_XH_04_Socket, symbol ESP32_Carrier:Conn_JST_XH_04_ENC
- added J15: BUZZER 5V, ESP32_Carrier:JST_XH_03_Socket, symbol ESP32_Carrier:GEN_JST_XH_03_Socket
- added J16: AOD4184 12V, ESP32_Carrier:JST_XH_04_Socket, symbol ESP32_Carrier:Conn_JST_XH_04_ENC
- added J18: EC11 ENC, ESP32_Carrier:JST_XH_04_Socket, symbol ESP32_Carrier:Conn_JST_XH_04_ENC
- added J8: HOME HOME1, ESP32_Carrier:JST_XH_02_Socket, symbol ESP32_Carrier:Conn_JST_XH_02
- added U5: ULN2003 A1, ESP32_Carrier:ULN2003_Module, symbol ESP32_Carrier:GEN_ULN2003_Module
- added U6: ULN2003 A2, ESP32_Carrier:ULN2003_Module, symbol ESP32_Carrier:GEN_ULN2003_Module
- added U7: ULN2003 A3, ESP32_Carrier:ULN2003_Module, symbol ESP32_Carrier:GEN_ULN2003_Module
- C21: value 100u/25V -> 220u/25V
- D2: value 1N5819 -> SS24
- J17: value TFT_LCD -> MSP3520 LCD
- J23: value TFT_TP -> MSP3520 TP
- U1: value ESP32_S3_DevKitC_1 -> ESP32-S3 DevKitC
- U2: value MP1584_5V3A -> MP1584 5V
Connections:
- net +12V: now also C24.1 (P1), C25.1 (P1), F1.2 (P2), J16.3 (ENC_A), U5.6 (P6), U6.6 (P6), U7.6 (P6)
- net +12V_RAW: now also D3.1 (P1)
- net +12V_SNS: now also C26.1 (P1), J10.2 (SNS), J12.2 (SNS), J14.1 (GND), J8.2 (SNS)
- net +3V3: now also J18.2 (3V3)
- net +5V: now also J15.1 (P1)
- net BLOWER: now also J16.1 (GND)
- net BLW_RET: now also J16.4 (ENC_B)
- net BUZZER: now also J15.3 (P3)
- net ENC_A: now also J18.3 (ENC_A)
- net ENC_B: now also J18.4 (ENC_B)
- net GND: now also C24.2 (P2), C25.2 (P2), C26.2 (P2), J14.2 (3V3), J15.2 (P2), J16.2 (3V3), J18.1 (GND), U5.5 (P5), U6.5 (P5), U7.5 (P5)
- net OPTO_IN1: now also J8.1 (SIG)
- net OPTO_IN2: now also J10.1 (SIG)
- net OPTO_IN3: now also J12.1 (SIG)
- net OPTO_IN4: now also J14.3 (ENC_A)
- net SR_Q0: now also U5.1 (P1)
- net SR_Q1: now also U5.2 (P2)
- net SR_Q10: now also U7.3 (P3)
- net SR_Q11: now also U7.4 (P4)
- net SR_Q2: now also U5.3 (P3)
- net SR_Q3: now also U5.4 (P4)
- net SR_Q4: now also U6.1 (P1)
- net SR_Q5: now also U6.2 (P2)
- net SR_Q6: now also U6.3 (P3)
- net SR_Q7: now also U6.4 (P4)
- net SR_Q8: now also U7.1 (P1)
- net SR_Q9: now also U7.2 (P2)
- new net +12V_PRE: D3.2 (P2), F1.1 (P1)
- no-connect marks 56 -> 32

Commit message: update BOM và PCB với danh sách linh kiện mới loại bỏ màn hình cảm ứng và động cơ điều chỉnh độ rộng vách thay bằng led 7 thanh và bàn phím dán
Parts:
- removed C10: 47u/25V, ESP32_Carrier:CP_Radial_D6_47u_25V, symbol ESP32_Carrier:GEN_CP_Radial_D6_47u_25V
- removed C20: 470u/25V, ESP32_Carrier:CP_Radial_D8_470u_25V, symbol ESP32_Carrier:GEN_CP_Radial_D8_470u_25V
- removed C21: 220u/25V, ESP32_Carrier:CP_Radial_D6_100u_25V, symbol ESP32_Carrier:GEN_CP_Radial_D6_100u_25V
- removed C25: 100n, ESP32_Carrier:C_0805_100n, symbol ESP32_Carrier:GEN_C_0805_100n
- removed D1: P6KE15A, ESP32_Carrier:Diode_TVS_DO41, symbol ESP32_Carrier:GEN_Diode_TVS_DO41
- removed D2: SS24, ESP32_Carrier:Diode_TVS_DO41, symbol ESP32_Carrier:GEN_Diode_TVS_DO41
- removed D3: SS54, ESP32_Carrier:Diode_TVS_DO41, symbol ESP32_Carrier:GEN_Diode_TVS_DO41
- removed J10: HOME HOME2, ESP32_Carrier:JST_XH_02_Socket, symbol ESP32_Carrier:Conn_JST_XH_02
- removed J12: HOME HOME3, ESP32_Carrier:JST_XH_02_Socket, symbol ESP32_Carrier:Conn_JST_XH_02
- removed J16: AOD4184 12V, ESP32_Carrier:JST_XH_04_Socket, symbol ESP32_Carrier:Conn_JST_XH_04_ENC
- removed J17: MSP3520 LCD, ESP32_Carrier:PinHeader_1x09_TFT_LCD, symbol ESP32_Carrier:Conn_1x09_TFT_LCD
- removed J18: EC11 ENC, ESP32_Carrier:JST_XH_04_Socket, symbol ESP32_Carrier:Conn_JST_XH_04_ENC
- removed J23: MSP3520 TP, ESP32_Carrier:PinHeader_1x05_TFT_TP, symbol ESP32_Carrier:Conn_1x05_TFT_TP
- removed J24: 595_CTRL, ESP32_Carrier:PinHeader_1x06_595CTRL, symbol ESP32_Carrier:GEN_PinHeader_1x06_595CTRL
- removed J25: 595_Q, ESP32_Carrier:PinHeader_1x24_595Q, symbol ESP32_Carrier:GEN_PinHeader_1x24_595Q
- removed J8: HOME HOME1, ESP32_Carrier:JST_XH_02_Socket, symbol ESP32_Carrier:Conn_JST_XH_02
- removed R1: 4k7, ESP32_Carrier:R_Axial_4k7_BUP, symbol ESP32_Carrier:R_BUP_Pullup
- removed R2, R3, R4, R45, R46, R47, R48: 10k, ESP32_Carrier:R_Axial_4k7_BUP, symbol ESP32_Carrier:R_BUP_Pullup
- removed R41, R42, R43, R44: 2k2, ESP32_Carrier:R_Axial_4k7_BUP, symbol ESP32_Carrier:R_BUP_Pullup
- removed U1: ESP32-S3 DevKitC, ESP32_Carrier:ESP32_S3_DevKitC_44Pin_Socket, symbol ESP32_Carrier:ESP32_S3_DevKitC_1
- removed U2: MP1584 5V, ESP32_Carrier:MP1584_5V3A, symbol ESP32_Carrier:MP1584_5V3A
- removed U41, U42, U43, U44: PC817, ESP32_Carrier:PC817_DIP4, symbol ESP32_Carrier:PC817_DIP4
- removed U5: ULN2003 A1, ESP32_Carrier:ULN2003_Module, symbol ESP32_Carrier:GEN_ULN2003_Module
- removed U6: ULN2003 A2, ESP32_Carrier:ULN2003_Module, symbol ESP32_Carrier:GEN_ULN2003_Module
- removed U7: ULN2003 A3, ESP32_Carrier:ULN2003_Module, symbol ESP32_Carrier:GEN_ULN2003_Module
- added BZ1: BUZZ, ESP32_Carrier:Buzzer_SMD_5V, symbol ESP32_Carrier:GEN_Buzzer_SMD_5V
- added C10: 47u/50V, ESP32_Carrier:CP_SMD_D6.3x5.8, symbol ESP32_Carrier:GEN_CP_SMD_D6_3x5_8
- added C20: 470u/50V, ESP32_Carrier:CP_SMD_D8x10, symbol ESP32_Carrier:GEN_CP_SMD_D8x10
- added C21: 220u/50V, ESP32_Carrier:CP_SMD_D6.3x5.8, symbol ESP32_Carrier:GEN_CP_SMD_D6_3x5_8
- added C3: 47u/10V, ESP32_Carrier:CP_SMD_D6.3x5.8, symbol ESP32_Carrier:GEN_CP_SMD_D6_3x5_8
- added C31, C51: 100n, ESP32_Carrier:C_0805_100n, symbol ESP32_Carrier:GEN_C_0805_100n
- added C5: 100u/16V, ESP32_Carrier:CP_SMD_D6.3x5.8, symbol ESP32_Carrier:GEN_CP_SMD_D6_3x5_8
- added Cbst: 10n, ESP32_Carrier:C_0805, symbol ESP32_Carrier:GEN_C_0805
- added Cc: 3n3, ESP32_Carrier:C_0805, symbol ESP32_Carrier:GEN_C_0805
- added D1: SMBJ26A, ESP32_Carrier:Diode_SMB_TVS, symbol ESP32_Carrier:GEN_Diode_SMB_TVS
- added D3: SS54, ESP32_Carrier:Diode_SMA, symbol ESP32_Carrier:GEN_Diode_SMA
- added D4: SS34, ESP32_Carrier:Diode_SMA, symbol ESP32_Carrier:GEN_Diode_SMA
- added J_DISP: 7SEG_EXT, ESP32_Carrier:PinHeader_1x10_7SEG, symbol ESP32_Carrier:GEN_PinHeader_1x10_7SEG
- added J_KEY: KEYPAD_EXT, ESP32_Carrier:PinHeader_1x08_Keypad, symbol ESP32_Carrier:GEN_PinHeader_1x08_Keypad
- added J_USB: USB, ESP32_Carrier:USB_MicroB, symbol ESP32_Carrier:GEN_USB_MicroB
- added L1: 10uH, ESP32_Carrier:L_SMD_6x6, symbol ESP32_Carrier:GEN_L_SMD_6x6
- added R1: 4k7, ESP32_Carrier:R_0805_4k7, symbol ESP32_Carrier:GEN_R_0805_4k7
- added R2, R48, Rfb2: 10k, ESP32_Carrier:R_0805_10k, symbol ESP32_Carrier:GEN_R_0805_10k
- added R44: 2k2, ESP32_Carrier:R_0805_2k2, symbol ESP32_Carrier:GEN_R_0805_2k2
- added Rfb1: 52k3, ESP32_Carrier:R_0805_4k7, symbol ESP32_Carrier:GEN_R_0805_4k7
- added U1: WROOM-32, ESP32_Carrier:ESP32_WROOM_32, symbol ESP32_Carrier:GEN_ESP32_WROOM_32
- added U2: MP1584EN, ESP32_Carrier:MP1584EN_SOT23-8, symbol ESP32_Carrier:GEN_MP1584EN_SOT23_8
- added U44: PC817, ESP32_Carrier:PC817_SOP4, symbol ESP32_Carrier:GEN_PC817_SOP4
- added U5: CH340C, ESP32_Carrier:CH340C, symbol ESP32_Carrier:GEN_CH340C
- added U6: AMS1117-3.3, ESP32_Carrier:AMS1117_SOT223, symbol ESP32_Carrier:GEN_AMS1117_SOT223
- added U7: TM1637, ESP32_Carrier:TM1637_SOP20, symbol ESP32_Carrier:GEN_TM1637_SOP20
- C26: value 100n SNS -> 100n
- F1: value 5x20 T3.15A -> T2.5A
- J1: value Screw_12V_IN -> 24V_IN
- J14: value BUP-30S -> BUP_U
- J15: value BUZZER 5V -> FIBER
- U3: value TMC2209 -> TMC_SOCK
Connections:
- net OPTO_IN4 is gone; now on net /OPTO_IN_BUP: J14.3 (ENC_A)
- net +3V3: now also C3.1 (P1), C31.1 (P1), R2.1 (P1), R48.1 (P1), U1.2 (P2), U1.3 (P3), U5.4 (P4), U6.2 (P2)
- net +5V: now also BZ1.1 (P1), C5.1 (P1), C51.1 (P1), J_USB.1 (P1), L1.2 (P2), Rfb1.1 (P1), U5.16 (P16), U6.3 (P3), U7.15 (P15); no longer J15.1 (P1)
- net GND: now also C10.2 (P2), C20.2 (P2), C21.2 (P2), C3.2 (P2), C31.2 (P2), C5.2 (P2), C51.2 (P2), Cc.2 (P2), D1.1 (P1), D4.1 (P1), J_USB.5 (P5), Rfb2.2 (P2), U1.1 (P1), U1.15 (P15), U1.20 (P20), U1.38 (P38), U2.5 (P5), U44.2 (P2), U44.3 (P3), U5.1 (P1), U6.1 (P1), U7.16 (P16)
- net +12V renamed +24V
- net +24V: now also C20.1 (P1), C21.1 (P1), D1.2 (P2), U2.2 (P2), U2.6 (P6)
- net +12V_PRE renamed +24V_PRE
- net +24V_PRE: now also D3.2 (P2)
- net +12V_RAW renamed +24V_RAW
- net +24V_RAW: now also D3.1 (P1)
- net +12V_SNS renamed +24V_SNS
- net +24V_SNS: now also J15.1 (P1), C10.1 (P1), R1.1 (P1), R44.1 (P1)
- net BUZZER renamed /OPTO_IN_BUP
- net /OPTO_IN_BUP: now also R1.2 (P2), R44.2 (P2), U44.1 (P1)
- net DIR renamed /DIR
- net /DIR: now also U1.28 (P28)
- net EN_TMC renamed /EN_TMC
- net /EN_TMC: now also R2.2 (P2), U1.30 (P30)
- net MotA1 renamed /MotA1
- net MotA2 renamed /MotA2
- net MotB1 renamed /MotB1
- net MotB2 renamed /MotB2
- net STEP renamed /STEP
- net /STEP: now also U1.27 (P27)
- new net /BUCK_BS: Cbst.1 (P1), U2.8 (P8)
- new net /BUCK_COMP: Cc.1 (P1), U2.3 (P3)
- new net /BUCK_FB: Rfb1.2 (P2), Rfb2.1 (P1), U2.4 (P4)
- new net /BUCK_SW: Cbst.2 (P2), D4.2 (P2), L1.1 (P1), U2.1 (P1)
- new net /BUP: R48.2 (P2), U1.26 (P26), U44.4 (P4)
- new net /BUZZER: BZ1.2 (P2), U1.10 (P10)
- new net /KEY_C0: J_KEY.5 (P5), U1.11 (P11)
- new net /KEY_C1: J_KEY.6 (P6), U1.9 (P9)
- new net /KEY_C2: J_KEY.7 (P7), U1.8 (P8)
- new net /KEY_C3: J_KEY.8 (P8), U1.29 (P29)
- new net /KEY_R0: J_KEY.1 (P1), U1.16 (P16)
- new net /KEY_R1: J_KEY.2 (P2), U1.14 (P14)
- new net /KEY_R2: J_KEY.3 (P3), U1.13 (P13)
- new net /KEY_R3: J_KEY.4 (P4), U1.12 (P12)
- new net /TM_CLK: U1.36 (P36), U7.18 (P18)
- new net /TM_DIO: U1.37 (P37), U7.17 (P17)
- new net /TM_G1: J_DISP.1 (P1), U7.1 (P1)
- new net /TM_G2: J_DISP.2 (P2), U7.2 (P2)
- new net /TM_G3: J_DISP.3 (P3), U7.3 (P3)
- new net /TM_SA: J_DISP.4 (P4), U7.7 (P7)
- new net /TM_SB: J_DISP.5 (P5), U7.8 (P8)
- new net /TM_SC: J_DISP.6 (P6), U7.9 (P9)
- new net /TM_SD: J_DISP.7 (P7), U7.10 (P10)
- new net /TM_SE: J_DISP.8 (P8), U7.11 (P11)
- new net /TM_SF: J_DISP.9 (P9), U7.12 (P12)
- new net /TM_SG: J_DISP.10 (P10), U7.13 (P13)
- new net /UART_RX: U1.34 (P34), U5.2 (P2)
- new net /UART_TX: U1.35 (P35), U5.3 (P3)
- new net /USB_DM: J_USB.2 (P2), U5.6 (P6)
- new net /USB_DP: J_USB.3 (P3), U5.5 (P5)
- no-connect marks 32 -> 38

Commit message: thay chip esp32 bằng stm32
Parts:
- removed BZ1: BUZZ, ESP32_Carrier:Buzzer_SMD_5V, symbol ESP32_Carrier:GEN_Buzzer_SMD_5V
- removed R10: 10R, ESP32_Carrier:R_1206_10R, symbol ESP32_Carrier:GEN_R_1206_10R
- removed U1: WROOM-32, ESP32_Carrier:ESP32_WROOM_32, symbol ESP32_Carrier:GEN_ESP32_WROOM_32
- added C20B: 220u/50V, ESP32_Carrier:CP_SMD_D6.3x5.8, symbol ESP32_Carrier:GEN_CP_SMD_D6_3x5_8
- added C24B, C52, C53, C_MCU, C_NRST: 100n, ESP32_Carrier:C_0805_100n, symbol ESP32_Carrier:GEN_C_0805_100n
- added C_MCU2: 1u, ESP32_Carrier:C_0805, symbol ESP32_Carrier:GEN_C_0805
- added C_XI, C_XO: 22p, ESP32_Carrier:C_0805, symbol ESP32_Carrier:GEN_C_0805
- added D5: SMBJ5.0A, ESP32_Carrier:Diode_SMB_TVS, symbol ESP32_Carrier:GEN_Diode_SMB_TVS
- added J_DBG: CortexDbg, ESP32_Carrier:Cortex_Debug_10, symbol ESP32_Carrier:GEN_Cortex_Debug_10
- added J_IN2: IN2, ESP32_Carrier:JST_XH_03_Socket, symbol ESP32_Carrier:GEN_JST_XH_03_Socket
- added J_IN3: IN3, ESP32_Carrier:JST_XH_03_Socket, symbol ESP32_Carrier:GEN_JST_XH_03_Socket
- added J_MOT1: MOT1, ESP32_Carrier:Mot_XH_04_Socket, symbol ESP32_Carrier:GEN_Mot_XH_04_Socket
- added J_MOT2: MOT2, ESP32_Carrier:Mot_XH_04_Socket, symbol ESP32_Carrier:GEN_Mot_XH_04_Socket
- added PTC_MOT, PTC_MOT2: 1.1A, ESP32_Carrier:PTC_1812, symbol ESP32_Carrier:GEN_PTC_1812
- added PTC_SNS: 0.2A, ESP32_Carrier:PTC_1812, symbol ESP32_Carrier:GEN_PTC_1812
- added R10: 22R, ESP32_Carrier:R_1206_22R, symbol ESP32_Carrier:GEN_R_1206_22R
- added R2B, R49, R50, R_BOOT, R_NRST, R_PWR_FLT, R_SWDIO, R_VIB_FLT: 10k, ESP32_Carrier:R_0805_10k, symbol ESP32_Carrier:GEN_R_0805_10k
- added R45, R46: 2k2, ESP32_Carrier:R_0805_2k2, symbol ESP32_Carrier:GEN_R_0805_2k2
- added SW_BOOT: BOOT0, ESP32_Carrier:SW_Push_6mm, symbol ESP32_Carrier:GEN_SW_Push_6mm
- added SW_NRST: NRST, ESP32_Carrier:SW_Push_6mm, symbol ESP32_Carrier:GEN_SW_Push_6mm
- added U1: STM32G030C8T6, ESP32_Carrier:STM32G030C8T6_LQFP48, symbol ESP32_Carrier:GEN_STM32G030C8T6_LQFP48
- added U4: TMC2, ESP32_Carrier:TMC2209_StepStick, symbol ESP32_Carrier:TMC2209_StepStick
- added U45, U46: PC817, ESP32_Carrier:PC817_SOP4, symbol ESP32_Carrier:GEN_PC817_SOP4
- added U_PWR: PWR_MOD, ESP32_Carrier:PowerMod_2CH_Sock, symbol ESP32_Carrier:GEN_PowerMod_2CH_Sock
- added U_VIB: VIB_SSR, ESP32_Carrier:VibAC_Sock, symbol ESP32_Carrier:GEN_VibAC_Sock
- added Y1: 12MHz, ESP32_Carrier:Crystal_SMD_3225, symbol ESP32_Carrier:GEN_Crystal_SMD_3225
- F1: value T2.5A -> T2A
- J_USB: value USB -> USB_MicroB
- U3: value TMC_SOCK -> TMC1
Connections:
- net +24V: now also PTC_MOT.1 (P1), PTC_MOT2.1 (P1), PTC_SNS.1 (P1), U_PWR.1 (P1), U_PWR.2 (P2), U_VIB.1 (P1); no longer C20.1 (P1), C24.1 (P1), U3.9 (VM)
- net +24V_SNS: now also J_IN2.1 (P1), J_IN3.1 (P1), R10.2 (P2), R45.1 (P1), R46.1 (P1)
- net +3V3: now also C52.1 (P1), C_MCU.1 (P1), C_MCU2.1 (P1), J_DBG.1 (P1), R2B.1 (P1), R49.1 (P1), R50.1 (P1), R_NRST.1 (P1), R_PWR_FLT.1 (P1), R_SWDIO.1 (P1), R_VIB_FLT.1 (P1), SW_BOOT.3 (P3), SW_BOOT.4 (P4), U1.4 (P4), U1.5 (P5), U1.6 (P6), U4.15 (VIO), U_PWR.5 (P5)
- net +5V: now also C53.1 (P1), D5.2 (P2)
- net /BUP: now also U1.14 (P14)
- net /DIR: now also U1.12 (P12)
- net /EN_TMC: now also U1.13 (P13)
- net /KEY_C0: now also U1.23 (P23)
- net /KEY_C1: now also U1.24 (P24)
- net /KEY_C2: now also U1.25 (P25)
- net /KEY_C3: now also U1.26 (P26)
- net /KEY_R0: now also U1.19 (P19)
- net /KEY_R1: now also U1.20 (P20)
- net /KEY_R2: now also U1.21 (P21)
- net /KEY_R3: now also U1.22 (P22)
- net /MotA1: now also J_MOT1.2 (P2)
- net /MotA2: now also J_MOT1.1 (P1)
- net /MotB1: now also J_MOT1.3 (P3)
- net /MotB2: now also J_MOT1.4 (P4)
- net /STEP: now also U1.11 (P11)
- net /TM_CLK: now also U1.15 (P15)
- net /TM_DIO: now also U1.16 (P16)
- net /UART_RX: now also U1.32 (P32)
- net /UART_TX: now also U1.29 (P29)
- net GND: now also C20B.2 (P2), C24B.2 (P2), C52.2 (P2), C53.2 (P2), C_MCU.2 (P2), C_MCU2.2 (P2), C_NRST.2 (P2), C_XI.2 (P2), C_XO.2 (P2), D5.1 (P1), J_DBG.3 (P3), J_DBG.5 (P5), J_DBG.8 (P8), J_DBG.9 (P9), J_IN2.2 (P2), J_IN3.2 (P2), R_BOOT.2 (P2), SW_NRST.3 (P3), SW_NRST.4 (P4), U1.7 (P7), U4.10 (GND), U4.16 (GND2), U45.2 (P2), U45.3 (P3), U46.2 (P2), U46.3 (P3), U_PWR.11 (P11), U_PWR.12 (P12), U_PWR.3 (P3), U_PWR.4 (P4), U_VIB.2 (P2), Y1.2 (P2), Y1.4 (P4)
- net /CH340_XI: now reaches U5.7 (P7)
- net /CH340_XI: now also C_XI.1 (P1), Y1.1 (P1)
- net /CH340_XO: now reaches U5.8 (P8)
- net /CH340_XO: now also C_XO.1 (P1), Y1.3 (P3)
- new net +24V_MOT: C20.1 (P1), C24.1 (P1), PTC_MOT.2 (P2), U3.9 (VM)
- new net +24V_MOT2: C20B.1 (P1), C24B.1 (P1), PTC_MOT2.2 (P2), U4.9 (VM)
- new net +24V_SNS_PRE: PTC_SNS.2 (P2), R10.1 (P1)
- new net /DIR2: U1.18 (P18), U4.8 (DIR)
- new net /EN_TMC2: R2B.2 (P2), U1.28 (P28), U4.1 (EN)
- new net /IN2: R49.2 (P2), U1.27 (P27), U45.4 (P4)
- new net /IN3: R50.2 (P2), U1.43 (P43), U46.4 (P4)
- new net /Mot2A1: J_MOT2.2 (P2), U4.12 (A1)
- new net /Mot2A2: J_MOT2.1 (P1), U4.11 (A2)
- new net /Mot2B1: J_MOT2.3 (P3), U4.13 (B1)
- new net /Mot2B2: J_MOT2.4 (P4), U4.14 (B2)
- new net /NRST: C_NRST.1 (P1), J_DBG.10 (P10), R_NRST.2 (P2), SW_NRST.1 (P1), SW_NRST.2 (P2), U1.10 (P10)
- new net /OPTO_IN2: J_IN2.3 (P3), R45.2 (P2), U45.1 (P1)
- new net /OPTO_IN3: J_IN3.3 (P3), R46.2 (P2), U46.1 (P1)
- new net /PWM_OUT1: U1.33 (P33), U_PWR.7 (P7)
- new net /PWM_OUT2: U1.34 (P34), U_PWR.8 (P8)
- new net /PWR_DIR: U1.45 (P45), U_PWR.10 (P10)
- new net /PWR_EN: U1.44 (P44), U_PWR.9 (P9)
- new net /PWR_FAULT: R_PWR_FLT.2 (P2), U1.46 (P46), U_PWR.6 (P6)
- new net /STEP2: U1.17 (P17), U4.7 (STEP)
- new net /SWCLK: J_DBG.4 (P4), R_BOOT.1 (P1), SW_BOOT.1 (P1), SW_BOOT.2 (P2), U1.36 (P36)
- new net /SWDIO: J_DBG.2 (P2), R_SWDIO.2 (P2), U1.35 (P35)
- new net /SWO: J_DBG.6 (P6), U1.42 (P42)
- new net /VIB_CTRL: U1.47 (P47), U_VIB.3 (P3)
- new net /VIB_FAULT: R_VIB_FLT.2 (P2), U1.48 (P48), U_VIB.4 (P4)
- no-connect marks 38 -> 39
