File: pcb/esp32_baseboard/esp32_baseboard.kicad_sch (KiCad schematic)
At the start: 73 parts, among them J1 24V_IN, J14 BUP_U, J15 FIBER, U1 STM32G030C8T6, U2 MP1584EN, U3 TMC1, U4 TMC2, U44 PC817, U45 PC817, U46 PC817, U5 CH340C, U6 AMS1117-3.3, U7 TM1637, Y1 12MHz

Commit message: Cập nhật carrier STM32: giắc N/S, USB+BOOT/RESET, courtyard ≥2.5mm.
Xóa pcb/esp32_soldered/.history và ignore thư mục .history.

Co-authored-by: Cursor <cursoragent@cursor.com>
Parts:
- removed J_DBG: CortexDbg, ESP32_Carrier:Cortex_Debug_10, symbol ESP32_Carrier:GEN_Cortex_Debug_10
- removed J_DISP: 7SEG_EXT, ESP32_Carrier:PinHeader_1x10_7SEG, symbol ESP32_Carrier:GEN_PinHeader_1x10_7SEG
- removed U7: TM1637, ESP32_Carrier:TM1637_SOP20, symbol ESP32_Carrier:GEN_TM1637_SOP20
- removed U_PWR: PWR_MOD, ESP32_Carrier:PowerMod_2CH_Sock, symbol ESP32_Carrier:GEN_PowerMod_2CH_Sock
- added C27: 100n, ESP32_Carrier:C_0805_100n, symbol ESP32_Carrier:GEN_C_0805_100n
- added J_CNT5: CNT5V, ESP32_Carrier:JST_XH_03_Socket, symbol ESP32_Carrier:GEN_JST_XH_03_Socket
- added J_DISP: TM1637_MOD, ESP32_Carrier:Disp_XH_04_Socket, symbol ESP32_Carrier:GEN_Disp_XH_04_Socket
- added J_P24N: P24_N, ESP32_Carrier:JST_XH_02_Socket, symbol ESP32_Carrier:Conn_JST_XH_02
- added J_P24S: P24_S, ESP32_Carrier:JST_XH_02_Socket, symbol ESP32_Carrier:Conn_JST_XH_02
- added J_P5N: P5_N, ESP32_Carrier:JST_XH_02_Socket, symbol ESP32_Carrier:Conn_JST_XH_02
- added R47: 1k, ESP32_Carrier:R_0805_1k, symbol ESP32_Carrier:GEN_R_0805_1k
- added R51: 10k, ESP32_Carrier:R_0805_10k, symbol ESP32_Carrier:GEN_R_0805_10k
- added U47: PC817, ESP32_Carrier:PC817_SOP4, symbol ESP32_Carrier:GEN_PC817_SOP4
- added U_PWR1: FET1, ESP32_Carrier:PowerMod_1CH_Sock, symbol ESP32_Carrier:GEN_PowerMod_1CH_Sock
- added U_PWR2: FET2, ESP32_Carrier:PowerMod_1CH_Sock, symbol ESP32_Carrier:GEN_PowerMod_1CH_Sock
Connections:
- net +24V: now also J_P24S.1 (SIG), U_PWR1.1 (P1), U_PWR2.1 (P1)
- net +24V_SNS: now also J_P24N.1 (SIG)
- net +3V3: now also R51.1 (P1), U_PWR1.3 (P3), U_PWR2.3 (P3)
- net +5V: now also C27.1 (P1), J_CNT5.1 (P1), J_DISP.3 (P3), J_P5N.1 (SIG), R47.1 (P1)
- net /PWM_OUT1: now also U_PWR1.4 (P4)
- net /PWM_OUT2: now also U_PWR2.4 (P4)
- net /PWR_FAULT: now also U_PWR1.6 (P6), U_PWR2.6 (P6)
- net /TM_CLK: now also J_DISP.1 (P1)
- net /TM_DIO: now also J_DISP.2 (P2)
- net GND: now also C27.2 (P2), J_CNT5.2 (P2), J_DISP.4 (P4), J_P24N.2 (SNS), J_P24S.2 (SNS), J_P5N.2 (SNS), U47.2 (P2), U47.3 (P3), U_PWR1.2 (P2), U_PWR2.2 (P2)
- net /CNT5: now reaches U1.39 (P39)
- net /CNT5: now also R51.2 (P2), U47.4 (P4)
- net /PWR_DIR renamed /PWR_EN2
- net /PWR_EN2: now also U_PWR2.5 (P5)
- net /PWR_EN renamed /PWR_EN1
- net /PWR_EN1: now also U_PWR1.5 (P5)
- net /SWO: no longer names the net of U1.42 (P42)
- new net /OPTO_IN_5V: J_CNT5.3 (P3), R47.2 (P2), U47.1 (P1)
- no-connect marks 39 -> 32
