File: pcb/esp32_baseboard/esp32_baseboard.kicad_sch (KiCad schematic)
At the start: 80 parts, among them J1 24V_IN, J14 BUP_U, J15 FIBER, U1 STM32G030C8T6, U2 MP1584EN, U3 TMC1, U4 TMC2, U44 PC817, U45 PC817, U46 PC817, U47 PC817, U5 CH340C, U6 AMS1117-3.3, Y1 12MHz

Commit message: update 3d view để khớp với PCB
Parts:
- J_DISP: value TM1637_MOD -> TM1637
- J_KEY: value KEYPAD_EXT -> KEYPAD
- J_USB: value USB_MicroB -> USB
- U1: value STM32G030C8T6 -> STM32G030
- U3: value TMC1 -> TMC2209
- U4: value TMC2 -> TMC2209
- U_PWR1: value FET1 -> MOSFET
- U_PWR2: value FET2 -> MOSFET
- U_VIB: value VIB_SSR -> SSR
