File: pcb/esp32_baseboard/esp32_baseboard.kicad_sch (KiCad schematic)
At the start: 80 parts, among them J1 24V_IN, J14 BUP_U, J15 FIBER, U1 STM32G030, U2 MP1584EN, U3 TMC2209, U4 TMC2209, U44 PC817, U45 PC817, U46 PC817, U47 PC817, U5 CH340C, U6 AMS1117-3.3, Y1 12MHz

Commit message: thêm review JLCPCB và cập nhật BOM, bỏ tracking JRE/out.
Co-authored-by: Cursor <cursoragent@cursor.com>
Parts:
- added C_V3: 100n, ESP32_Carrier:C_0805_100n, symbol ESP32_Carrier:GEN_C_0805_100n
- added R_FREQ: 100k, ESP32_Carrier:R_0805_100k, symbol ESP32_Carrier:GEN_R_0805_100k
- added R_PD_DIR, R_PD_DIR2, R_PD_EN1, R_PD_EN2, R_PD_PWM1, R_PD_PWM2, R_PD_STEP, R_PD_STEP2, R_PD_VIB: 10k, ESP32_Carrier:R_0805_10k, symbol ESP32_Carrier:GEN_R_0805_10k
- C10: footprint ESP32_Carrier:CP_SMD_D6.3x5.8 -> ESP32_Carrier:CP_SMD_D6.3x8
- C20B, C21: value 220u/50V -> 47u/50V; footprint ESP32_Carrier:CP_SMD_D6.3x5.8 -> ESP32_Carrier:CP_SMD_D6.3x8
- C3: value 47u/10V -> 47u/50V; footprint ESP32_Carrier:CP_SMD_D6.3x5.8 -> ESP32_Carrier:CP_SMD_D6.3x8
- F1: value T2A -> FUSE T2A
- J1: value 24V_IN -> 24V IN
- J14: value BUP_U -> COUNT
- J_CNT5: value CNT5V -> COUNT 5V
- J_DISP: value TM1637 -> DISPLAY
- J_IN2: value IN2 -> IN 2
- J_IN3: value IN3 -> IN 3
- J_MOT1: value MOT1 -> MOTOR 1
- J_MOT2: value MOT2 -> MOTOR 2
- J_P24N: value P24_N -> 24V SNS
- J_P24S: value P24_S -> 24V AUX
- J_P5N: value P5_N -> +5V OUT
- SW_BOOT: value BOOT0 -> BOOT; footprint ESP32_Carrier:SW_Push_6mm -> ESP32_Carrier:SW_Push_6mm_SMD
- SW_NRST: value NRST -> RESET; footprint ESP32_Carrier:SW_Push_6mm -> ESP32_Carrier:SW_Push_6mm_SMD
- U2: footprint ESP32_Carrier:MP1584EN_SOT23-8 -> ESP32_Carrier:MP1584EN_SOIC-8-EP
- U3: value TMC2209 -> TMC1
- U4: value TMC2209 -> TMC2
- U_PWR1: value MOSFET -> MOSFET 1
- U_PWR2: value MOSFET -> MOSFET 2
- U_VIB: value SSR -> VIB SSR
Connections:
- net +24V: now also U2.7 (P7); no longer U2.2 (P2), U2.6 (P6)
- net +3V3: now also U6.TAB; no longer U5.4 (P4)
- net /DIR: now also R_PD_DIR.1 (P1)
- net /DIR2: now also R_PD_DIR2.1 (P1)
- net /PWM_OUT1: now also R_PD_PWM1.1 (P1)
- net /PWM_OUT2: now also R_PD_PWM2.1 (P1)
- net /PWR_EN1: now also R_PD_EN1.1 (P1)
- net /PWR_EN2: now also R_PD_EN2.1 (P1)
- net /STEP: now also R_PD_STEP.1 (P1)
- net /STEP2: now also R_PD_STEP2.1 (P1)
- net /VIB_CTRL: now also R_PD_VIB.1 (P1)
- net GND: now also J_USB.MH1 (SHIELD), J_USB.MH2 (SHIELD), U2.9 (EP), C_V3.2 (P2), R_FREQ.2 (P2), R_PD_DIR.2 (P2), R_PD_DIR2.2 (P2), R_PD_EN1.2 (P2), R_PD_EN2.2 (P2), R_PD_PWM1.2 (P2), R_PD_PWM2.2 (P2), R_PD_STEP.2 (P2), R_PD_STEP2.2 (P2), R_PD_VIB.2 (P2)
- new net /BUCK_FREQ: R_FREQ.1 (P1), U2.6 (P6)
- new net /CH340_V3: C_V3.1 (P1), U5.4 (P4)
Other:
- note added: "24V IN / SNS"
- note added: "3V3"
- note added: "BUCK +5V"
- note added: "DO / VIB"
- note added: "HMI"
- note added: "MCU STM32G030"
- note added: "OPTO IN"
- note added: "TMC1"
- note added: "TMC2"
- note added: "USB-UART"
