File: pcb/STM32G030C8T6/STM32G030C8T6.kicad_pcb (KiCad board)
At the start: 2 copper layers, 150 x 100 mm, 93 parts, among them J1 24V IN, J14 COUNT, J15 FIBER, U1 STM32G030, U2 MP1584EN, U3 TMC1, U4 TMC2, U44 PC817, U45 PC817, U46 PC817, U47 PC817, U5 CH340C, U6 AMS1117-3.3, Y1 12MHz

Commit message: thêm đèn led báo trạng thái và thêm kịch bản review cho pcb
Parts:
- added D_LED24: LED_AMB, STM32G030C8T6:LED_0805, F.Cu at (182.0, 58.0)
- added D_LED3V3: LED_GRN, STM32G030C8T6:LED_0805, F.Cu at (182.0, 61.2)
- added D_LEDBUP: LED_YEL, STM32G030C8T6:LED_0805, F.Cu at (116.0, 72.0)
- added D_LEDCNT5: LED_YEL, STM32G030C8T6:LED_0805, F.Cu at (116.0, 75.2)
- added D_LEDERR: LED_RED, STM32G030C8T6:LED_0805, F.Cu at (182.0, 67.6)
- added D_LEDIN2: LED_YEL, STM32G030C8T6:LED_0805, F.Cu at (116.0, 78.4)
- added D_LEDIN3: LED_YEL, STM32G030C8T6:LED_0805, F.Cu at (116.0, 81.6)
- added D_LEDRUN: LED_GRN, STM32G030C8T6:LED_0805, F.Cu at (182.0, 64.4)
- added R_LED24: 2k2, STM32G030C8T6:R_0805_2k2, F.Cu at (178.0, 58.0)
- added R_LED33: 1k, STM32G030C8T6:R_0805_1k, F.Cu at (178.0, 61.2)
- added R_LEDBUP: 1k, STM32G030C8T6:R_0805_1k, F.Cu at (112.0, 72.0)
- added R_LEDCNT5: 1k, STM32G030C8T6:R_0805_1k, F.Cu at (112.0, 75.2)
- added R_LEDERR: 1k, STM32G030C8T6:R_0805_1k, F.Cu at (178.0, 67.6)
- added R_LEDIN2: 1k, STM32G030C8T6:R_0805_1k, F.Cu at (112.0, 78.4)
- added R_LEDIN3: 1k, STM32G030C8T6:R_0805_1k, F.Cu at (112.0, 81.6)
- added R_LEDRUN: 1k, STM32G030C8T6:R_0805_1k, F.Cu at (178.0, 64.4)
Connections:
- U1 pad 21: unconnected-(U1-21-Pad21) -> /LED_RUN
- U1 pad 30: unconnected-(U1-30-Pad30) -> /LED_ERR
Other:
- board text added: "24V"
- board text added: "3V3"
- board text added: "BUP"
- board text added: "CNT5"
- board text added: "ERR"
- board text added: "IN2"
- board text added: "IN3"
- board text added: "RUN"
- board text added: "SNS LED"
- board text added: "STATUS"

Commit message: thay đổi giắc điều khiển máng rung sang on/off phù hợp máy việt nam
Parts:
- removed R_PD_EN1, R_PD_EN2, R_PD_PWM1, R_PD_PWM2, R_PD_VIB, R_PWR_FLT, R_VIB_FLT: 10k, STM32G030C8T6:R_0805_10k
- removed U_PWR1: MOSFET 1, STM32G030C8T6:PowerMod_1CH_Sock
- removed U_PWR2: MOSFET 2, STM32G030C8T6:PowerMod_1CH_Sock
- removed U_VIB: VIB SSR, STM32G030C8T6:VibAC_Sock
- added D_DO1: SS24, STM32G030C8T6:Diode_SMA, F.Cu at (136.0, 138.0)
- added D_DO2: SS24, STM32G030C8T6:Diode_SMA, F.Cu at (155.0, 138.0)
- added J_DO1: DO1, STM32G030C8T6:JST_XH_03_Socket, F.Cu at (131.1, 147.6)
- added J_DO2: DO2, STM32G030C8T6:JST_XH_03_Socket, F.Cu at (150.0, 147.6)
- added Q_DO1: AO3400, STM32G030C8T6:MOSFET_SOT23, F.Cu at (131.0, 138.0)
- added Q_DO2: AO3400, STM32G030C8T6:MOSFET_SOT23, F.Cu at (150.0, 138.0)
- added R_DO1: 1k, STM32G030C8T6:R_0805_1k, F.Cu at (159.6, 137.0)
- added R_DO2: 1k, STM32G030C8T6:R_0805_1k, F.Cu at (167.1, 138.0)
- added R_PD_DO1: 10k, STM32G030C8T6:R_0805_10k, F.Cu at (147.4, 132.5)
- added R_PD_DO2: 10k, STM32G030C8T6:R_0805_10k, F.Cu at (154.6, 137.0)
- J1: value 24V IN -> 24V_IN
- J14: value COUNT -> BUP_U
- J_CNT5: value COUNT 5V -> CNT5V
- J_DISP: value DISPLAY -> TM1637
- J_IN2: value IN 2 -> IN2
- J_IN3: value IN 3 -> IN3
- J_MOT1: value MOTOR 1 -> MOT1
- J_MOT2: value MOTOR 2 -> MOT2
- J_P24S: value 24V AUX -> P24_S
- SW_BOOT: value BOOT -> BOOT0
- SW_NRST: value RESET -> NRST
- U3: value TMC1 -> TMC2209
- U4: value TMC2 -> TMC2209
- moved D_LEDIN2 66.6 mm to (180.0, 60.0)
- moved R_LEDIN2 66.6 mm to (176.0, 60.0)
- moved R_LEDCNT5 65.8 mm to (176.0, 60.0)
- moved D_LEDIN3 65.2 mm to (176.0, 56.0)
- moved R_LEDBUP 64.5 mm to (176.0, 64.0)
- moved R_LEDIN3 63.3 mm to (168.0, 52.0)
- moved D_LEDCNT5 63.0 mm to (176.0, 56.0)
- moved D_LEDBUP 58.2 mm to (172.0, 56.0)
- moved D_LEDERR 15.9 mm to (168.0, 60.0)
- moved R_LEDERR 15.3 mm to (168.0, 56.0)
- moved D_LED24 10.2 mm to (172.0, 56.0)
- moved R_LED24 6.32 mm to (172.0, 60.0)
- moved D_LED3V3 6.12 mm to (176.0, 60.0)
- moved R_LED33 6.12 mm to (172.0, 60.0)
- moved R_LEDRUN 4.83 mm to (176.0, 60.0)
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Connections:
- J_USB pad 4: unconnected-(J_USB-4-Pad4) -> (no net)
- U1 pad 1: unconnected-(U1-1-Pad1) -> (no net)
- U1 pad 2: unconnected-(U1-2-Pad2) -> (no net)
- U1 pad 22: /PWM_OUT1 -> /DO1
- U1 pad 23: /PWM_OUT2 -> /DO2
- U1 pad 24: /PWR_EN1 -> (no net)
- U1 pad 25: /PWR_EN2 -> (no net)
- U1 pad 26: /PWR_FAULT -> (no net)
- U1 pad 27: /VIB_CTRL -> (no net)
- U1 pad 28: /VIB_FAULT -> (no net)
- U1 pad 3: unconnected-(U1-3-Pad3) -> (no net)
- U1 pad 31: unconnected-(U1-31-Pad31) -> (no net)
- U1 pad 33: unconnected-(U1-33-Pad33) -> (no net)
- U1 pad 34: unconnected-(U1-34-Pad34) -> (no net)
- U1 pad 39: unconnected-(U1-39-Pad39) -> (no net)
- U1 pad 40: unconnected-(U1-40-Pad40) -> (no net)
- U1 pad 8: unconnected-(U1-8-Pad8) -> (no net)
- U1 pad 9: unconnected-(U1-9-Pad9) -> (no net)
- U2 pad 2: unconnected-(U2-2-Pad2) -> (no net)
- U3 pad 2: unconnected-(U3-MS1-Pad2) -> (no net)
- U3 pad 3: unconnected-(U3-MS2-Pad3) -> (no net)
- U3 pad 4: unconnected-(U3-PDN-Pad4) -> (no net)
- U3 pad 5: unconnected-(U3-PDN2-Pad5) -> (no net)
- U3 pad 6: unconnected-(U3-CLK-Pad6) -> (no net)
- U4 pad 2: unconnected-(U4-MS1-Pad2) -> (no net)
- U4 pad 3: unconnected-(U4-MS2-Pad3) -> (no net)
- U4 pad 4: unconnected-(U4-PDN-Pad4) -> (no net)
- U4 pad 5: unconnected-(U4-PDN2-Pad5) -> (no net)
- U4 pad 6: unconnected-(U4-CLK-Pad6) -> (no net)
- U5 pad 10: unconnected-(U5-10-Pad10) -> (no net)
- U5 pad 11: unconnected-(U5-11-Pad11) -> (no net)
- U5 pad 12: unconnected-(U5-12-Pad12) -> (no net)
- U5 pad 13: unconnected-(U5-13-Pad13) -> (no net)
- U5 pad 14: unconnected-(U5-14-Pad14) -> (no net)
- U5 pad 15: unconnected-(U5-15-Pad15) -> (no net)
- U5 pad 9: unconnected-(U5-9-Pad9) -> (no net)
Routing:
- net /PWR_FAULT: track 110.7 -> 0.00 mm
- net /VIB_FAULT: track 91.5 -> 0.00 mm
- net /PWR_EN1: track 90.5 -> 0.00 mm, vias 2 -> 0
- net /VIB_CTRL: track 88.1 -> 0.00 mm
- net /PWM_OUT1: track 86.1 -> 0.00 mm
- net /PWR_EN2: track 84.6 -> 0.00 mm
- net /PWM_OUT2: track 81.8 -> 0.00 mm
Other:
- board text added: "N: SNS/HMI/USB | S: J1 MOT1 MOT2 DO1 DO2 P24 | TMC inland"
- board text removed: "24V"
- board text removed: "3V3"
- board text removed: "BUP"
- board text removed: "CNT5"
- board text removed: "ERR"
- board text removed: "IN2"
- board text removed: "IN3"
- board text removed: "N: SNS/HMI/USB | S: J1 MOT1 MOT2 PWR1 PWR2 VIB P24 | TMC inland"
- board text removed: "RUN"
- board text removed: "SNS LED"
- board text removed: "STATUS"
