File: pcb/STM32G030C8T6/STM32G030C8T6.kicad_sch (KiCad schematic)
At the start: 89 parts, among them J1 24V IN, J14 COUNT, J15 FIBER, U1 STM32G030, U2 MP1584EN, U3 TMC1, U4 TMC2, U44 PC817, U45 PC817, U46 PC817, U47 PC817, U5 CH340C, U6 AMS1117-3.3, Y1 12MHz

Commit message: thay đổi giắc điều khiển máng rung sang on/off phù hợp máy việt nam
Parts:
- removed R_PD_EN1, R_PD_EN2, R_PD_PWM1, R_PD_PWM2, R_PD_VIB, R_PWR_FLT, R_VIB_FLT: 10k, STM32G030C8T6:R_0805_10k, symbol STM32G030C8T6:GEN_R_0805_10k
- removed U_PWR1: MOSFET 1, STM32G030C8T6:PowerMod_1CH_Sock, symbol STM32G030C8T6:GEN_PowerMod_1CH_Sock
- removed U_PWR2: MOSFET 2, STM32G030C8T6:PowerMod_1CH_Sock, symbol STM32G030C8T6:GEN_PowerMod_1CH_Sock
- removed U_VIB: VIB SSR, STM32G030C8T6:VibAC_Sock, symbol STM32G030C8T6:GEN_VibAC_Sock
- added D_DO1, D_DO2: SS24, STM32G030C8T6:Diode_SMA, symbol STM32G030C8T6:GEN_Diode_SMA
- added D_LED24: LED_AMB, STM32G030C8T6:LED_0805, symbol STM32G030C8T6:GEN_LED_0805
- added D_LED3V3, D_LEDRUN: LED_GRN, STM32G030C8T6:LED_0805, symbol STM32G030C8T6:GEN_LED_0805
- added D_LEDBUP, D_LEDCNT5, D_LEDIN2, D_LEDIN3: LED_YEL, STM32G030C8T6:LED_0805, symbol STM32G030C8T6:GEN_LED_0805
- added D_LEDERR: LED_RED, STM32G030C8T6:LED_0805, symbol STM32G030C8T6:GEN_LED_0805
- added J_DO1: DO1, STM32G030C8T6:JST_XH_03_Socket, symbol STM32G030C8T6:GEN_JST_XH_03_Socket
- added J_DO2: DO2, STM32G030C8T6:JST_XH_03_Socket, symbol STM32G030C8T6:GEN_JST_XH_03_Socket
- added Q_DO1, Q_DO2: AO3400, STM32G030C8T6:MOSFET_SOT23, symbol STM32G030C8T6:GEN_MOSFET_SOT23
- added R_DO1, R_DO2, R_LED33, R_LEDBUP, R_LEDCNT5, R_LEDERR, R_LEDIN2, R_LEDIN3, R_LEDRUN: 1k, STM32G030C8T6:R_0805_1k, symbol STM32G030C8T6:GEN_R_0805_1k
- added R_LED24: 2k2, STM32G030C8T6:R_0805_2k2, symbol STM32G030C8T6:GEN_R_0805_2k2
- added R_PD_DO1, R_PD_DO2: 10k, STM32G030C8T6:R_0805_10k, symbol STM32G030C8T6:GEN_R_0805_10k
- J1: value 24V IN -> 24V_IN
- J14: value COUNT -> BUP_U
- J_CNT5: value COUNT 5V -> CNT5V
- J_DISP: value DISPLAY -> TM1637
- J_IN2: value IN 2 -> IN2
- J_IN3: value IN 3 -> IN3
- J_MOT1: value MOTOR 1 -> MOT1
- J_MOT2: value MOTOR 2 -> MOT2
- J_P24S: value 24V AUX -> P24_S
- SW_BOOT: value BOOT -> BOOT0
- SW_NRST: value RESET -> NRST
- U3: value TMC1 -> TMC2209
- U4: value TMC2 -> TMC2209
Connections:
- net +24V: now also D_DO1.2, D_DO2.2, J_DO1.1, J_DO2.1, R_LED24.1
- net +3V3: now also R_LED33.1, R_LEDBUP.1, R_LEDCNT5.1, R_LEDIN2.1, R_LEDIN3.1
- net /BUP: now also D_LEDBUP.2
- net /CNT5: now also D_LEDCNT5.2
- net /IN2: now also D_LEDIN2.2
- net /IN3: now also D_LEDIN3.2
- net GND: now also D_LED24.2, D_LED3V3.2, D_LEDERR.2, D_LEDRUN.2, J_DO1.2, J_DO2.2, Q_DO1.2, Q_DO2.2, R_PD_DO1.2, R_PD_DO2.2
- net /LED_RUN: now reaches U1.21
- net /LED_RUN: now also R_LEDRUN.1
- net /LED_ERR: now reaches U1.30
- net /LED_ERR: now also R_LEDERR.1
- net /PWM_OUT1 renamed /DO1
- net /DO1: now also R_DO1.1, R_PD_DO1.1
- net /PWM_OUT2 renamed /DO2
- net /DO2: now also R_DO2.1, R_PD_DO2.1
- net /PWR_EN1: no longer names the net of U1.24
- net /PWR_EN2: no longer names the net of U1.25
- net /PWR_FAULT: no longer names the net of U1.26
- net /VIB_CTRL: no longer names the net of U1.27
- net /VIB_FAULT: no longer names the net of U1.28
- new net /DO1_G: Q_DO1.1, R_DO1.2
- new net /DO1_OUT: D_DO1.1, J_DO1.3, Q_DO1.3
- new net /DO2_G: Q_DO2.1, R_DO2.2
- new net /DO2_OUT: D_DO2.1, J_DO2.3, Q_DO2.3
- new net /LED24_A: D_LED24.1, R_LED24.2
- new net /LED33_A: D_LED3V3.1, R_LED33.2
- new net /LEDBUP_A: D_LEDBUP.1, R_LEDBUP.2
- new net /LEDCNT5_A: D_LEDCNT5.1, R_LEDCNT5.2
- new net /LEDERR_A: D_LEDERR.1, R_LEDERR.2
- new net /LEDIN2_A: D_LEDIN2.1, R_LEDIN2.2
- new net /LEDIN3_A: D_LEDIN3.1, R_LEDIN3.2
- new net /LEDRUN_A: D_LEDRUN.1, R_LEDRUN.2
- no-connect marks 31 -> 34
